Commit message: robot_description

File: scout_ws/src/robot_description/urdf/mobile_robot/scout_v2.urdf.xacro (robot description, xacro)
@@ -32,5 +32,5 @@
 				<geometry>
 					<mesh
-						filename="file://$(find agilex_scout)/meshes/mobile_robot/mobile_robot_base_link.dae" />
+						filename="file://$(find robot_description)/meshes/mobile_robot/mobile_robot_base_link.dae" />
 				</geometry>
 			</visual>
@@ -64,6 +64,6 @@
 		</joint>
 		<!-- Scout wheel macros -->
-		<xacro:include filename="$(find agilex_scout)/urdf/mobile_robot/scout_wheel_type1.xacro" />
-		<xacro:include filename="$(find agilex_scout)/urdf/mobile_robot/scout_wheel_type2.xacro" />
+		<xacro:include filename="$(find robot_description)/urdf/mobile_robot/scout_wheel_type1.xacro" />
+		<xacro:include filename="$(find robot_description)/urdf/mobile_robot/scout_wheel_type2.xacro" />
 		<!-- wheel labeled from 0 to 3, conter-clockwise, starting from front right wheel -->
 		<!-- motor 1 and 2 (left side) are mechanically installed in a reversed direction -->
@@ -90,5 +90,5 @@
 		<!-- Gazebo definitions  -->
 		<xacro:if value="${load_gazebo}">
-			<xacro:include filename="$(find agilex_scout)/urdf/mobile_robot/scout_v2.gazebo" />
+			<xacro:include filename="$(find robot_description)/urdf/mobile_robot/scout_v2.gazebo" />
 		</xacro:if>
 	</xacro:macro>

File: scout_ws/src/robot_description/urdf/mobile_robot/scout_wheel_type1.xacro (robot description, xacro)
@@ -24,5 +24,5 @@
 -->
 <robot xmlns:xacro="http://ros.org/wiki/xacro" name="scout_v2">
-	<xacro:macro name="scout_wheel_type2" params="wheel_prefix x y z phi">
+	<xacro:macro name="scout_wheel_type1" params="wheel_prefix x y z phi">
 		<link name="${wheel_prefix}_wheel_link">
 			<inertial>
@@ -34,5 +34,5 @@
 				<origin xyz="0 0 0" rpy="0 0 0" />
 				<geometry>
-					<mesh filename="file://$(find agilex_scout)/meshes/mobile_robot/wheel_type2.dae" />
+					<mesh filename="file://$(find robot_description)/meshes/mobile_robot/wheel_type1.dae" />
 				</geometry>
 			</visual>

File: scout_ws/src/robot_description/urdf/mobile_robot/scout_wheel_type2.xacro (robot description, xacro)
@@ -24,5 +24,5 @@
 -->
 <robot xmlns:xacro="http://ros.org/wiki/xacro" name="scout_v2">
-	<xacro:macro name="scout_wheel_type1" params="wheel_prefix x y z phi">
+	<xacro:macro name="scout_wheel_type2" params="wheel_prefix x y z phi">
 		<link name="${wheel_prefix}_wheel_link">
 			<inertial>
@@ -34,5 +34,5 @@
 				<origin xyz="0 0 0" rpy="0 0 0" />
 				<geometry>
-					<mesh filename="file://$(find agilex_scout)/meshes/mobile_robot/wheel_type1.dae" />
+					<mesh filename="file://$(find robot_description)/meshes/mobile_robot/wheel_type2.dae" />
 				</geometry>
 			</visual>

File: scout_ws/src/robot_description/urdf/robot.urdf.xacro (robot description, xacro)
@@ -6,9 +6,9 @@
 	<xacro:arg name="load_gazebo" default="true" />
 	<xacro:arg name="simulation" default="true" />
-	<xacro:include filename="$(find agilex_scout)/urdf/mobile_robot/scout_v2.urdf.xacro" />
+	<xacro:include filename="$(find robot_description)/urdf/mobile_robot/scout_v2.urdf.xacro" />
 	<xacro:scout_v2 odometry_source="$(arg odometry_source)" load_gazebo="$(arg load_gazebo)" />
 	<xacro:unless value="$(arg simulation)">
 		<!-- addition of OS1 sensor when loading the real Scout -->
-		<xacro:include filename="$(find agilex_scout)/urdf/sensors/os1.urdf" />
+		<xacro:include filename="$(find robot_description)/urdf/sensors/os1.urdf" />
 		<joint name="os1_joint" type="fixed">
 			<origin xyz="0.2 0.0 0.64" rpy="0.0 0.0 0.0" />

File: scout_ws/src/robot_description/urdf/sensors/os1.urdf (robot description, URDF)
Before this commit: robot os1_description, 1 links, 0 joints
Links:
- link os_sensor: geometry visual mesh filename=file://$(find robot_description)/meshes/sensors/laser_link.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 scale=1.0 1.0 1.0
